File: PCB/Sensor_Luz/Sensor_Luz.kicad_pcb (KiCad board)
At the start: 2 copper layers, 12 parts, among them J1 Conn_02x20_Odd_Even, J2 Conn_02x20_Odd_Even, J3 Conn_01x02_Male, J4 Conn_01x04_Female, J5 Conn_01x02_Male, J6 Conn_01x06_Female, J7 Conn_01x02_Male, Q1 BC817

Commit message: PCB actualizado
Parts:
- added C1: 0.1uF, Capacitor_THT:C_Disc_D5.0mm_W2.5mm_P2.50mm, F.Cu at (84.0, 93.0)
- added C2: 0.33uF, Capacitor_THT:C_Disc_D5.0mm_W2.5mm_P2.50mm, F.Cu at (84.0, 102.5)
- added J8: Conn_01x02_Male, Connector_PinSocket_2.54mm:PinSocket_1x02_P2.54mm_Vertical, F.Cu at (129.0, 78.0)
- added U1: LM7805_TO220, Package_TO_SOT_THT:TO-220-3_Vertical, F.Cu at (77.9, 100.8)
- moved J3 22.1 mm to (79.0, 70.0)
- moved J4 16.1 mm to (129.0, 99.0), turned to 180 degrees
- moved R1 10.0 mm to (75.7, 109.6)
- moved R3 10.0 mm to (81.3, 109.6)
- moved R2 8.06 mm to (75.7, 113.9)
- moved R4 8.06 mm to (81.3, 113.9)
- moved J5 7.81 mm to (85.0, 81.5), turned to 0 degrees
- moved J6 6.61 mm to (129.0, 118.0)
- moved Q1 5.10 mm to (78.0, 120.0)
- moved J7 4.07 mm to (76.0, 81.5), turned to 0 degrees
- moved J1 1.00 mm to (65.5, 72.0)
- moved J2 1.00 mm to (137.0, 72.0)
Connections:
- J2 pad 17: +5V -> /VDDA
- J3 pad 1: +9V -> Net-(C1-Pad1)
- J4 pad 2: /I2C_SDA -> GND
- J4 pad 4: GND -> /I2C_SDA
Routing:
- net Net-(C1-Pad1): track 0.00 -> 39.2 mm
- net /CH1: track 92.3 -> 70.5 mm
- net +5V: track 0.00 -> 20.2 mm, vias 0 -> 2
- net +9V: track 14.4 -> 33.5 mm
- net /VDDA: track 0.00 -> 16.1 mm
- net +3V3: track 40.8 -> 51.0 mm
- net /232_RX: track 13.2 -> 18.6 mm
- net /232_TX: track 13.8 -> 18.6 mm
- net /I2C_SDA: track 14.1 -> 9.44 mm
- net /GPIO1: track 14.9 -> 10.3 mm
- net /I2C_SCL: track 14.0 -> 10.0 mm
- net Net-(Q1-Pad3): track 9.13 -> 6.03 mm
- net Net-(Q1-Pad1): track 7.70 -> 4.67 mm
- net Net-(J5-Pad1): track 7.00 -> 9.00 mm

Commit message: PCB actualizado y hoja de datos
Parts:
- added D1: 1N4148W, Diode_SMD:D_SOD-123, F.Cu at (81.0, 111.7)
- added Q2: BC807, Package_TO_SOT_SMD:SOT-23, F.Cu at (88.0, 120.0)
- added R5: 4.7k, Resistor_SMD:R_0805_2012Metric, F.Cu at (88.0, 109.1)
- C1, C2, U1: moved to B.Cu
- R2: value 10k -> 100k
- moved C2 18.2 mm to (79.0, 85.0), turned to 180 degrees
- moved U1 17.3 mm to (85.0, 85.0)
- moved J5 14.8 mm to (88.0, 96.0)
- moved J7 14.7 mm to (78.0, 96.0)
- moved C1 13.9 mm to (79.0, 80.0), turned to 180 degrees
- moved R3 8.05 mm to (88.0, 114.1), turned to 90 degrees
- moved R4 5.07 mm to (81.1, 119.0), turned to 180 degrees
- moved J6 3.62 mm to (129.0, 121.6)
- moved Q1 2.00 mm to (76.0, 120.0)
Connections:
- R3 pad 1: +9V -> Net-(Q2-Pad3)
- R4 pad 1: /CH1 -> Net-(D1-Pad1)
Routing:
- net Net-(C1-Pad1): track 39.2 -> 6.03 mm
- net +9V: track 33.5 -> 51.4 mm, vias 0 -> 2
- net Net-(D1-Pad1): track 0.00 -> 11.1 mm
- net /CH1: track 70.5 -> 62.1 mm
- net Net-(Q2-Pad3): track 0.00 -> 5.36 mm
- net +3V3: track 51.0 -> 55.3 mm
- net /232_TX: track 18.6 -> 22.5 mm
- net /232_RX: track 18.6 -> 21.5 mm
- net Net-(Q1-Pad3): track 6.03 -> 3.52 mm
- net Net-(J5-Pad1): track 9.00 -> 10.0 mm

Commit message: Cambio PCB
Parts:
- removed D1: 1N4148W, Diode_SMD:D_SOD-123
- Q1: value BC817 -> BC548; footprint Package_TO_SOT_SMD:SOT-23 -> Package_TO_SOT_THT:TO-92_Inline
- Q2: value BC807 -> BC558; footprint Package_TO_SOT_SMD:SOT-23 -> Package_TO_SOT_THT:TO-92_Inline
- R1: value 330 -> 330k; footprint Resistor_SMD:R_0805_2012Metric -> Resistor_THT:R_Axial_DIN0204_L3.6mm_D1.6mm_P7.62mm_Horizontal
- R2, R4: footprint Resistor_SMD:R_0805_2012Metric -> Resistor_THT:R_Axial_DIN0204_L3.6mm_D1.6mm_P7.62mm_Horizontal
- R3: value 10K -> 47K; footprint Resistor_SMD:R_0805_2012Metric -> Resistor_THT:R_Axial_DIN0204_L3.6mm_D1.6mm_P7.62mm_Horizontal
- R5: value 4.7k -> 22k; footprint Resistor_SMD:R_0805_2012Metric -> Resistor_THT:R_Axial_DIN0204_L3.6mm_D1.6mm_P7.62mm_Horizontal
- moved R4 13.0 mm to (81.0, 106.0), turned to 270 degrees
- moved Q2 11.4 mm to (88.0, 108.5), turned to 90 degrees
- moved R1 4.85 mm to (73.0, 113.6), turned to 90 degrees
- moved R5 4.43 mm to (89.0, 113.4), turned to 270 degrees
- moved R3 3.08 mm to (85.0, 113.4), turned to 270 degrees
- moved Q1 2.00 mm to (78.0, 120.0), turned to 180 degrees
- moved R2 1.35 mm to (77.0, 113.6)
Connections:
- Q1 pad 2: GND -> Net-(Q1-Pad2)
- Q1 pad 3: Net-(Q1-Pad3) -> GND
- Q2 pad 1: Net-(D1-Pad1) -> Net-(Q2-Pad1)
- Q2 pad 2: +9V -> Net-(Q2-Pad2)
- Q2 pad 3: Net-(Q2-Pad3) -> +9V
- R2 pad 1: Net-(Q1-Pad1) -> Net-(Q1-Pad2)
- R3 pad 1: Net-(Q2-Pad3) -> Net-(Q2-Pad1)
- R4 pad 1: Net-(D1-Pad1) -> Net-(Q2-Pad2)
- R4 pad 2: Net-(Q1-Pad3) -> Net-(Q1-Pad1)
Routing:
- net +9V: track 51.4 -> 37.1 mm, vias 2 -> 0
- net Net-(D1-Pad1): track 11.1 -> 0.00 mm
- net Net-(C1-Pad1): track 6.03 -> 16.0 mm
- net Net-(Q2-Pad2): track 0.00 -> 7.53 mm
- net /CH1: track 62.1 -> 68.6 mm
- net Net-(Q1-Pad2): track 0.00 -> 6.49 mm
- net Net-(Q2-Pad1): track 0.00 -> 6.08 mm
- net Net-(Q2-Pad3): track 5.36 -> 0.00 mm
- net Net-(Q1-Pad1): track 4.41 -> 8.37 mm
- net Net-(Q1-Pad3): track 3.52 -> 0.00 mm
- net /GPIO1: track 10.3 -> 11.3 mm
