File: PCB/Sensor_Luz/Sensor_Luz.sch (KiCad schematic (older format))
At the start: 12 parts, among them J1 Conn_02x20_Odd_Even, J2 Conn_02x20_Odd_Even, J3 Conn_01x02_Male, J4 Conn_01x04_Female, J5 Conn_01x02_Male, J6 Conn_01x06_Female, J7 Conn_01x02_Male, Q1 BC817

Commit message: PCB actualizado
Parts:
- added C1: 0.1uF, Capacitor_THT:C_Disc_D5.0mm_W2.5mm_P2.50mm, symbol Device:C
- added C2: 0.33uF, Capacitor_THT:C_Disc_D5.0mm_W2.5mm_P2.50mm, symbol Device:C
- added J8: Conn_01x02_Male, Connector_PinSocket_2.54mm:PinSocket_1x02_P2.54mm_Vertical, symbol Connector:Conn_01x02_Male
- added U1: LM7805_TO220, Package_TO_SOT_THT:TO-220-3_Vertical, symbol Regulator_Linear:LM7805_TO220
Connections:
- net +5V: now also J8.1 (Pin_1); no longer J2.17 (Pin_17)
- net +9V: now also C2.1, U1.1 (VI); no longer J3.1 (Pin_1)
- net GND: now also J4.2 (Pin_2), C1.2, C2.2, U1.2 (GND); no longer J4.4 (Pin_4)
- net I2C_SDA: now also J4.4 (Pin_4); no longer J4.2 (Pin_2)
- new net: C1.1, J3.1 (Pin_1), U1.3 (VO)
- new net VDDA: J2.17 (Pin_17), J8.2 (Pin_2)
Other:
- moved on the sheet: J2, J3, J4, J5, J6, J7, Q1, R1, R2, R3, R4

Commit message: PCB actualizado y hoja de datos
Parts:
- added D1: 1N4148W, Diode_SMD:D_SOD-123, symbol Diode:1N4148W
- added Q2: BC807, Package_TO_SOT_SMD:SOT-23, symbol Transistor_BJT:BC807
- added R5: 4.7k, Resistor_SMD:R_0805_2012Metric, symbol Device:R
- R2: value 10k -> 100k
Connections:
- net +9V: now also D1.2 (A), Q2.2 (E); no longer R3.1
- net CH1: now also R5.1; no longer R4.1
- net GND: now also R5.2
- new net: Q2.3 (C), R3.1
- new net: D1.1 (K), Q2.1 (B), R4.1
- no-connect marks 38 -> 44
Other:
- moved on the sheet: J5, J7, J8, R3
Changed lines of the file:
@@
 L Device:R R3
 U 1 1 5DB5ECB6
-P 4050 4650
-F 0 "R3" H 4120 4696 50  0000 L CNN
-F 1 "10K" H 4120 4605 50  0000 L CNN
-F 2 "Resistor_SMD:R_0805_2012Metric" V 3980 4650 50  0001 C CNN
-F 3 "~" H 4050 4650 50  0001 C CNN
-	1    4050 4650
+P 4850 5350
+F 0 "R3" H 4920 5396 50  0000 L CNN
+F 1 "10K" H 4920 5305 50  0000 L CNN
+F 2 "Resistor_SMD:R_0805_2012Metric" V 4780 5350 50  0001 C CNN
+F 3 "~" H 4850 5350 50  0001 C CNN
+	1    4850 5350
 	1    0    0    -1
 $EndComp
@@
 P 3500 5500
 F 0 "R2" V 3293 5500 50  0000 C CNN
-F 1 "10k" V 3384 5500 50  0000 C CNN
+F 1 "100k" V 3384 5500 50  0000 C CNN
 F 2 "Resistor_SMD:R_0805_2012Metric" V 3430 5500 50  0001 C CNN
 F 3 "~" H 3500 5500 50  0001 C CNN
@@
 	4050 5200 4050 5300
 Wire Wire Line
-	4050 4900 4050 4850
-Wire Wire Line
 	3750 5500 3650 5500
 Wire Wire Line
@@
 L Connector:Conn_01x02_Male J5
 U 1 1 5DC57AAA
-P 5250 4400
-F 0 "J5" H 5222 4374 50  0000 R CNN
-F 1 "Conn_01x02_Male" H 5222 4283 50  0000 R CNN
-F 2 "Connector_PinSocket_2.54mm:PinSocket_1x02_P2.54mm_Vertical" H 5250 4400 50  0001 C CNN
-F 3 "~" H 5250 4400 50  0001 C CNN
-	1    5250 4400
+P 9600 2350
+F 0 "J5" H 9572 2324 50  0000 R CNN
+F 1 "Conn_01x02_Male" H 9572 2233 50  0000 R CNN
+F 2 "Connector_PinSocket_2.54mm:PinSocket_1x02_P2.54mm_Vertical" H 9600 2350 50  0001 C CNN
+F 3 "~" H 9600 2350 50  0001 C CNN
+	1    9600 2350
 	-1   0    0    -1
 $EndComp
@@
 Wire Wire Line
 	4050 4400 4050 4500
-Wire Wire Line
-	4550 4400 4050 4400
 $Comp
 L power:GND #PWR010
@@
 L power:GND #PWR013
 U 1 1 5DC6457F
-P 5000 4550
-F 0 "#PWR013" H 5000 4300 50  0001 C CNN
-F 1 "GND" H 5005 4377 50  0000 C CNN
-F 2 "" H 5000 4550 50  0001 C CNN
-F 3 "" H 5000 4550 50  0001 C CNN
-	1    5000 4550
-	1    0    0    -1
-$EndComp
-Wire Wire Line
-	5000 4550 5000 4500
-Wire Wire Line
-	5000 4500 5050 4500
+P 9350 2500
+F 0 "#PWR013" H 9350 2250 50  0001 C CNN
+F 1 "GND" H 9355 2327 50  0000 C CNN
+F 2 "" H 9350 2500 50  0001 C CNN
+F 3 "" H 9350 2500 50  0001 C CNN
+	1    9350 2500
+	1    0    0    -1
+$EndComp
+Wire Wire Line
+	9350 2500 9350 2450
+Wire Wire Line
+	9350 2450 9400 2450
 Wire Wire Line
 	2000 4500 2050 4500
-Text Label 3750 4850 0    50   ~ 0
+Text Label 5100 5550 0    50   ~ 0
 CH1
 Text Label 2950 5500 0    50   ~ 0
 GPIO1
 Wire Wire Line
-	3750 4850 4050 4850
-Connection ~ 4050 4850
-Wire Wire Line
-	4050 4850 4050 4800
-Wire Wire Line
 	2950 5500 3250 5500
 Connection ~ 3250 5500
@@
 L power:+5V #PWR04
 U 1 1 5DC811AD
-P 3700 2000
-F 0 "#PWR04" H 3700 1850 50  0001 C CNN
-F 1 "+5V" H 3715 2173 50  0000 C CNN
-F 2 "" H 3700 2000 50  0001 C CNN
-F 3 "" H 3700 2000 50  0001 C CNN
-	1    3700 2000
+P 8500 1700
+F 0 "#PWR04" H 8500 1550 50  0001 C CNN
+F 1 "+5V" H 8515 1873 50  0000 C CNN
+F 2 "" H 8500 1700 50  0001 C CNN
+F 3 "" H 8500 1700 50  0001 C CNN
+	1    8500 1700
 	1    0    0    -1
 $EndComp
@@
 NoConn ~ 3950 1850
 NoConn ~ 3950 1950
-NoConn ~ 3950 2050
 NoConn ~ 3950 2150
 NoConn ~ 4900 1650
@@
 L Connector:Conn_01x02_Male J7
 U 1 1 5DBA020A
-P 4650 4200
-F 0 "J7" V 4712 4244 50  0000 L CNN
-F 1 "Conn_01x02_Male" V 4550 3900 50  0000 L CNN
-F 2 "Connector_PinSocket_2.54mm:PinSocket_1x02_P2.54mm_Vertical" H 4650 4200 50  0001 C CNN
-F 3 "~" H 4650 4200 50  0001 C CNN
-	1    4650 4200
-	0    1    1    0
-$EndComp
-Wire Wire Line
-	4650 4400 5050 4400
+P 9600 2000
+F 0 "J7" H 9500 2000 50  0000 L CNN
+F 1 "Conn_01x02_Male" H 8950 2100 50  0000 L CNN
+F 2 "Connector_PinSocket_2.54mm:PinSocket_1x02_P2.54mm_Vertical" H 9600 2000 50  0001 C CNN
+F 3 "~" H 9600 2000 50  0001 C CNN
+	1    9600 2000
+	-1   0    0    1
+$EndComp
 $Comp
 L Connector_Generic:Conn_02x20_Odd_Even J1
@@
 L Connector:Conn_01x02_Male J8
 U 1 1 5DC60556
-P 3200 2150
-F 0 "J8" H 3308 2331 50  0000 C CNN
-F 1 "Conn_01x02_Male" H 3308 2240 50  0000 C CNN
-F 2 "Connector_PinSocket_2.54mm:PinSocket_1x02_P2.54mm_Vertical" H 3200 2150 50  0001 C CNN
-F 3 "~" H 3200 2150 50  0001 C CNN
-	1    3200 2150
-	1    0    0    -1
-$EndComp
-Wire Wire Line
-	3400 2250 4300 2250
-Wire Wire Line
-	3400 2150 3700 2150
-Wire Wire Line
-	3700 2150 3700 2000
+P 8000 1850
+F 0 "J8" H 8108 2031 50  0000 C CNN
+F 1 "Conn_01x02_Male" H 8108 1940 50  0000 C CNN
+F 2 "Connector_PinSocket_2.54mm:PinSocket_1x02_P2.54mm_Vertical" H 8000 1850 50  0001 C CNN
+F 3 "~" H 8000 1850 50  0001 C CNN
+	1    8000 1850
+	1    0    0    -1
+$EndComp
+Wire Wire Line
+	8200 1850 8500 1850
+Wire Wire Line
+	8500 1850 8500 1700
 Wire Wire Line
 	6000 2000 6350 2000
@@
 Wire Wire Line
 	5900 1800 6350 1800
+Wire Wire Line
+	9400 2350 9350 2350
+Wire Wire Line
+	9350 2350 9350 2000
+Wire Wire Line
+	9350 2000 9400 2000
+$Comp
+L power:+9V #PWR016
+U 1 1 5DD6B004
+P 9350 1850
+F 0 "#PWR016" H 9350 1700 50  0001 C CNN
+F 1 "+9V" H 9365 2023 50  0000 C CNN
+F 2 "" H 9350 1850 50  0001 C CNN
+F 3 "" H 9350 1850 50  0001 C CNN
+	1    9350 1850
+	1    0    0    -1
+$EndComp
+Wire Wire Line
+	9350 1850 9350 1900
+Wire Wire Line
+	9350 1900 9400 1900
+Wire Wire Line
+	4050 4800 4050 4850
+$Comp
+L Diode:1N4148W D1
+U 1 1 5DD73588
+P 4050 4650
+F 0 "D1" V 4096 4570 50  0000 R CNN
+F 1 "1N4148W" V 4005 4570 50  0000 R CNN
+F 2 "Diode_SMD:D_SOD-123" H 4050 4475 50  0001 C CNN
+F 3 "https://www.vishay.com/docs/85748/1n4148w.pdf" H 4050 4650 50  0001 C CNN
+	1    4050 4650
+	0    -1   -1   0
+$EndComp
+$Comp
+L Transistor_BJT:BC807 Q2
+U 1 1 5DD74ACB
+P 4750 4850
+F 0 "Q2" H 4941 4804 50  0000 L CNN
+F 1 "BC807" H 4941 4895 50  0000 L CNN
+F 2 "Package_TO_SOT_SMD:SOT-23" H 4950 4775 50  0001 L CIN
+F 3 "http://www.fairchildsemi.com/ds/BC/BC807.pdf" H 4750 4850 50  0001 L CNN
+	1    4750 4850
+	1    0    0    1
+$EndComp
+$Comp
+L Device:R R5
+U 1 1 5DD8D747
+P 4850 5750
+F 0 "R5" H 4920 5796 50  0000 L CNN
+F 1 "4.7k" H 4920 5705 50  0000 L CNN
+F 2 "Resistor_SMD:R_0805_2012Metric" V 4780 5750 50  0001 C CNN
+F 3 "~" H 4850 5750 50  0001 C CNN
+	1    4850 5750
+	1    0    0    -1
+$EndComp
+Wire Wire Line
+	4850 5600 4850 5550
+Wire Wire Line
+	4850 5200 4850 5050
+Wire Wire Line
+	4850 4650 4850 4400
+Wire Wire Line
+	4850 4400 4050 4400
+Wire Wire Line
+	4550 4850 4050 4850
+Connection ~ 4050 4850
+Wire Wire Line
+	4050 4850 4050 4900
+Wire Wire Line
+	4850 5900 4850 5950
+Wire Wire Line
+	4850 5950 4050 5950
+Wire Wire Line
+	4850 5550 5100 5550
+Connection ~ 4850 5550
+Wire Wire Line
+	4850 5550 4850 5500
+Wire Wire Line
+	3950 2250 4300 2250
+Text Label 8500 1950 0    50   ~ 0
+VDDA
+Wire Wire Line
+	8500 1950 8200 1950
+NoConn ~ 3950 3350
+NoConn ~ 3950 3250
+NoConn ~ 3950 3150
+NoConn ~ 3950 3050
+NoConn ~ 3950 2950
+NoConn ~ 3950 2850
+NoConn ~ 3950 2750
 $EndSCHEMATC

Commit message: Cambio PCB
Parts:
- removed D1: 1N4148W, Diode_SMD:D_SOD-123, symbol Diode:1N4148W
- removed Q1: BC817, Package_TO_SOT_SMD:SOT-23, symbol Transistor_BJT:BC817
- removed Q2: BC807, Package_TO_SOT_SMD:SOT-23, symbol Transistor_BJT:BC807
- added Q1: BC548, Package_TO_SOT_THT:TO-92_Inline, symbol Transistor_BJT:BC548
- added Q2: BC558, Package_TO_SOT_THT:TO-92_Inline, symbol Transistor_BJT:BC558
- R1: value 330 -> 330k; footprint Resistor_SMD:R_0805_2012Metric -> Resistor_THT:R_Axial_DIN0204_L3.6mm_D1.6mm_P7.62mm_Horizontal
- R2, R4: footprint Resistor_SMD:R_0805_2012Metric -> Resistor_THT:R_Axial_DIN0204_L3.6mm_D1.6mm_P7.62mm_Horizontal
- R3: value 10K -> 47K; footprint Resistor_SMD:R_0805_2012Metric -> Resistor_THT:R_Axial_DIN0204_L3.6mm_D1.6mm_P7.62mm_Horizontal
- R5: value 4.7k -> 22k; footprint Resistor_SMD:R_0805_2012Metric -> Resistor_THT:R_Axial_DIN0204_L3.6mm_D1.6mm_P7.62mm_Horizontal
Connections:
- net +9V: now also Q2.3 (E)
- net GND: now also Q1.3 (E)
- net at R3.1: now also Q2.1 (C)
- net at R4.1: now also Q2.2 (B)
- net at R4.2: now also Q1.1 (C)
- net at R2.1: now also Q1.2 (B)
Other:
- moved on the sheet: C1, C2, J2, J3, J5, J6, J7, R1, R2, R3, R4, R5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
